File: hw/pcb/TrueStrike42.kicad_pcb (KiCad board)
At the start: 2 copper layers, 101 parts, among them U1 ProMicro, U2 74HC4051, U3 74HC4051, U4 74HC4051, U5 74HC4051, U6 74HC4051, U7 74HC4051, U8 74HC4051, U9 74HC4051

Commit message: Update TrueStrike42.kicad_pcb
Parts:
- moved C44 101.2 mm to (108.0, 49.2), turned to 90 degrees
- moved C45 99.7 mm to (108.0, 68.3), turned to 90 degrees
- moved C43 99.5 mm to (108.0, 30.2), turned to 90 degrees
- moved U2 96.4 mm to (108.0, 38.9)
- moved U3 96.4 mm to (108.0, 57.9)
- moved U4 96.4 mm to (108.0, 77.0)
- moved C47 96.0 mm to (185.7, 49.2), turned to 90 degrees
- moved C46 95.7 mm to (185.7, 30.2), turned to 90 degrees
- moved C48 94.6 mm to (185.7, 68.3), turned to 90 degrees
- moved U5 92.1 mm to (185.6, 38.9)
- moved U6 92.1 mm to (185.7, 57.9)
- moved U7 92.1 mm to (185.7, 77.0)
- moved C11 1.47 mm to (93.7, 54.0)
- moved C17 1.47 mm to (93.7, 73.0)
- moved C38 1.47 mm to (93.7, 92.1)
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
Commit message: Update PCB and schematic
Parts:
- added C51: 1uF, Capacitor_SMD:C_0805_2012Metric_Pad1.18x1.45mm_HandSolder, B.Cu at (22.2, 51.6)
- added C52: 1uF, Capacitor_SMD:C_0805_2012Metric_Pad1.18x1.45mm_HandSolder, B.Cu at (41.3, 46.8)
- added C53: 1uF, Capacitor_SMD:C_0805_2012Metric_Pad1.18x1.45mm_HandSolder, B.Cu at (60.3, 37.3)
- added C54: 1uF, Capacitor_SMD:C_0805_2012Metric_Pad1.18x1.45mm_HandSolder, B.Cu at (79.4, 32.5)
- added C55: 1uF, Capacitor_SMD:C_0805_2012Metric_Pad1.18x1.45mm_HandSolder, B.Cu at (98.4, 38.9)
- added C56: 1uF, Capacitor_SMD:C_0805_2012Metric_Pad1.18x1.45mm_HandSolder, B.Cu at (117.5, 38.9)
- added C57: 1uF, Capacitor_SMD:C_0805_2012Metric_Pad1.18x1.45mm_HandSolder, B.Cu at (22.2, 70.6)
- added C58: 1uF, Capacitor_SMD:C_0805_2012Metric_Pad1.18x1.45mm_HandSolder, B.Cu at (41.3, 65.9)
- added C59: 1uF, Capacitor_SMD:C_0805_2012Metric_Pad1.18x1.45mm_HandSolder, B.Cu at (60.3, 56.4)
- added C60: 1uF, Capacitor_SMD:C_0805_2012Metric_Pad1.18x1.45mm_HandSolder, B.Cu at (79.4, 51.6)
- added C61: 1uF, Capacitor_SMD:C_0805_2012Metric_Pad1.18x1.45mm_HandSolder, B.Cu at (98.4, 57.9)
- added C62: 1uF, Capacitor_SMD:C_0805_2012Metric_Pad1.18x1.45mm_HandSolder, B.Cu at (117.5, 57.9)
- added C63: 1uF, Capacitor_SMD:C_0805_2012Metric_Pad1.18x1.45mm_HandSolder, B.Cu at (117.5, 77.0)
- added C64: 1uF, Capacitor_SMD:C_0805_2012Metric_Pad1.18x1.45mm_HandSolder, B.Cu at (98.4, 77.0)
- added C65: 1uF, Capacitor_SMD:C_0805_2012Metric_Pad1.18x1.45mm_HandSolder, B.Cu at (79.4, 70.6)
- added C66: 1uF, Capacitor_SMD:C_0805_2012Metric_Pad1.18x1.45mm_HandSolder, B.Cu at (60.3, 75.4)
- added C67: 1uF, Capacitor_SMD:C_0805_2012Metric_Pad1.18x1.45mm_HandSolder, B.Cu at (41.3, 84.9)
- added C68: 1uF, Capacitor_SMD:C_0805_2012Metric_Pad1.18x1.45mm_HandSolder, B.Cu at (22.2, 89.7)
- added C69: 1uF, Capacitor_SMD:C_0805_2012Metric_Pad1.18x1.45mm_HandSolder, B.Cu at (79.4, 96.0)
- added C70: 1uF, Capacitor_SMD:C_0805_2012Metric_Pad1.18x1.45mm_HandSolder, B.Cu at (98.4, 96.0)
- added C71: 1uF, Capacitor_SMD:C_0805_2012Metric_Pad1.18x1.45mm_HandSolder, B.Cu at (127.0, 100.8)
- added C72: 1uF, Capacitor_SMD:C_0805_2012Metric_Pad1.18x1.45mm_HandSolder, B.Cu at (166.7, 100.8)
- added C73: 1uF, Capacitor_SMD:C_0805_2012Metric_Pad1.18x1.45mm_HandSolder, B.Cu at (195.3, 96.0)
- added C74: 1uF, Capacitor_SMD:C_0805_2012Metric_Pad1.18x1.45mm_HandSolder, B.Cu at (214.3, 96.0)
- added C75: 1uF, Capacitor_SMD:C_0805_2012Metric_Pad1.18x1.45mm_HandSolder, B.Cu at (271.5, 89.7)
- added C76: 1uF, Capacitor_SMD:C_0805_2012Metric_Pad1.18x1.45mm_HandSolder, B.Cu at (252.4, 84.9)
- added C77: 1uF, Capacitor_SMD:C_0805_2012Metric_Pad1.18x1.45mm_HandSolder, B.Cu at (233.4, 75.4)
- added C78: 1uF, Capacitor_SMD:C_0805_2012Metric_Pad1.18x1.45mm_HandSolder, B.Cu at (214.3, 70.6)
- added C79: 1uF, Capacitor_SMD:C_0805_2012Metric_Pad1.18x1.45mm_HandSolder, B.Cu at (195.3, 77.0)
- added C80: 1uF, Capacitor_SMD:C_0805_2012Metric_Pad1.18x1.45mm_HandSolder, B.Cu at (176.2, 77.0)
- added C81: 1uF, Capacitor_SMD:C_0805_2012Metric_Pad1.18x1.45mm_HandSolder, B.Cu at (176.2, 57.9)
- added C82: 1uF, Capacitor_SMD:C_0805_2012Metric_Pad1.18x1.45mm_HandSolder, B.Cu at (195.3, 57.9)
- added C83: 1uF, Capacitor_SMD:C_0805_2012Metric_Pad1.18x1.45mm_HandSolder, B.Cu at (214.3, 51.6)
- added C84: 1uF, Capacitor_SMD:C_0805_2012Metric_Pad1.18x1.45mm_HandSolder, B.Cu at (233.4, 56.4)
- added C85: 1uF, Capacitor_SMD:C_0805_2012Metric_Pad1.18x1.45mm_HandSolder, B.Cu at (252.4, 65.9)
- added C86: 1uF, Capacitor_SMD:C_0805_2012Metric_Pad1.18x1.45mm_HandSolder, B.Cu at (271.5, 70.6)
- added C87: 1uF, Capacitor_SMD:C_0805_2012Metric_Pad1.18x1.45mm_HandSolder, B.Cu at (271.5, 51.6)
- added C88: 1uF, Capacitor_SMD:C_0805_2012Metric_Pad1.18x1.45mm_HandSolder, B.Cu at (252.4, 46.8)
- added C89: 1uF, Capacitor_SMD:C_0805_2012Metric_Pad1.18x1.45mm_HandSolder, B.Cu at (233.4, 37.3)
- added C90: 1uF, Capacitor_SMD:C_0805_2012Metric_Pad1.18x1.45mm_HandSolder, B.Cu at (214.3, 32.5)
- added C91: 1uF, Capacitor_SMD:C_0805_2012Metric_Pad1.18x1.45mm_HandSolder, B.Cu at (195.3, 38.9)
- added C92: 1uF, Capacitor_SMD:C_0805_2012Metric_Pad1.18x1.45mm_HandSolder, B.Cu at (176.2, 38.9)
- added C93: 1uF, Capacitor_SMD:C_0805_2012Metric_Pad1.18x1.45mm_HandSolder, B.Cu at (131.0, 46.0)
- added D1: SK6812MINI-E, project-specific-library:SK6812MINI-E_nusumi, B.Cu at (117.5, 34.1)
- added D10: SK6812MINI-E, project-specific-library:SK6812MINI-E_nusumi_Rotated, B.Cu at (79.4, 46.8)
- added D11: SK6812MINI-E, project-specific-library:SK6812MINI-E_nusumi_Rotated, B.Cu at (98.4, 53.2)
- added D12: SK6812MINI-E, project-specific-library:SK6812MINI-E_nusumi_Rotated, B.Cu at (117.5, 53.2)
- added D13: SK6812MINI-E, project-specific-library:SK6812MINI-E_nusumi, B.Cu at (117.5, 72.2)
- added D14: SK6812MINI-E, project-specific-library:SK6812MINI-E_nusumi, B.Cu at (98.4, 72.2)
- added D15: SK6812MINI-E, project-specific-library:SK6812MINI-E_nusumi, B.Cu at (79.4, 65.9)
- added D16: SK6812MINI-E, project-specific-library:SK6812MINI-E_nusumi, B.Cu at (60.3, 70.6)
- added D17: SK6812MINI-E, project-specific-library:SK6812MINI-E_nusumi, B.Cu at (41.3, 80.2)
- added D18: SK6812MINI-E, project-specific-library:SK6812MINI-E_nusumi, B.Cu at (22.2, 84.9)
- added D19: SK6812MINI-E, project-specific-library:SK6812MINI-E_nusumi_Rotated, B.Cu at (79.4, 91.3)
- added D2: SK6812MINI-E, project-specific-library:SK6812MINI-E_nusumi, B.Cu at (98.4, 34.1)
- added D20: SK6812MINI-E, project-specific-library:SK6812MINI-E_nusumi_Rotated, B.Cu at (98.4, 91.3)
- added D21: SK6812MINI-E, project-specific-library:SK6812MINI-E_nusumi_Rotated, B.Cu at (127.0, 96.0)
- added D22: SK6812MINI-E, project-specific-library:SK6812MINI-E_nusumi_Rotated, B.Cu at (166.7, 96.0)
- added D23: SK6812MINI-E, project-specific-library:SK6812MINI-E_nusumi_Rotated, B.Cu at (195.3, 91.3)
- added D24: SK6812MINI-E, project-specific-library:SK6812MINI-E_nusumi_Rotated, B.Cu at (214.3, 91.3)
- added D25: SK6812MINI-E, project-specific-library:SK6812MINI-E_nusumi, B.Cu at (271.5, 84.9)
- added D26: SK6812MINI-E, project-specific-library:SK6812MINI-E_nusumi, B.Cu at (252.4, 80.2)
- added D27: SK6812MINI-E, project-specific-library:SK6812MINI-E_nusumi, B.Cu at (233.4, 70.6)
- added D28: SK6812MINI-E, project-specific-library:SK6812MINI-E_nusumi, B.Cu at (214.3, 65.9)
- added D29: SK6812MINI-E, project-specific-library:SK6812MINI-E_nusumi, B.Cu at (195.3, 72.2)
- added D3: SK6812MINI-E, project-specific-library:SK6812MINI-E_nusumi, B.Cu at (79.4, 27.8)
- added D30: SK6812MINI-E, project-specific-library:SK6812MINI-E_nusumi, B.Cu at (176.2, 72.2)
- added D31: SK6812MINI-E, project-specific-library:SK6812MINI-E_nusumi_Rotated, B.Cu at (176.2, 53.2)
- added D32: SK6812MINI-E, project-specific-library:SK6812MINI-E_nusumi_Rotated, B.Cu at (195.3, 53.2)
- added D33: SK6812MINI-E, project-specific-library:SK6812MINI-E_nusumi_Rotated, B.Cu at (214.3, 46.8)
- added D34: SK6812MINI-E, project-specific-library:SK6812MINI-E_nusumi_Rotated, B.Cu at (233.4, 51.6)
- added D35: SK6812MINI-E, project-specific-library:SK6812MINI-E_nusumi_Rotated, B.Cu at (252.4, 61.1)
- added D36: SK6812MINI-E, project-specific-library:SK6812MINI-E_nusumi_Rotated, B.Cu at (271.5, 65.9)
- added D37: SK6812MINI-E, project-specific-library:SK6812MINI-E_nusumi, B.Cu at (271.5, 46.8)
- added D38: SK6812MINI-E, project-specific-library:SK6812MINI-E_nusumi, B.Cu at (252.4, 42.1)
- added D39: SK6812MINI-E, project-specific-library:SK6812MINI-E_nusumi, B.Cu at (233.4, 32.5)
- added D4: SK6812MINI-E, project-specific-library:SK6812MINI-E_nusumi, B.Cu at (60.3, 32.5)
- added D40: SK6812MINI-E, project-specific-library:SK6812MINI-E_nusumi, B.Cu at (214.3, 27.8)
- added D41: SK6812MINI-E, project-specific-library:SK6812MINI-E_nusumi, B.Cu at (195.3, 34.1)
- added D42: SK6812MINI-E, project-specific-library:SK6812MINI-E_nusumi, B.Cu at (176.2, 34.1)
- added D5: SK6812MINI-E, project-specific-library:SK6812MINI-E_nusumi, B.Cu at (41.3, 42.1)
- added D6: SK6812MINI-E, project-specific-library:SK6812MINI-E_nusumi, B.Cu at (22.2, 46.8)
- added D7: SK6812MINI-E, project-specific-library:SK6812MINI-E_nusumi_Rotated, B.Cu at (22.2, 65.9)
- added D8: SK6812MINI-E, project-specific-library:SK6812MINI-E_nusumi_Rotated, B.Cu at (41.3, 61.1)
- added D9: SK6812MINI-E, project-specific-library:SK6812MINI-E_nusumi_Rotated, B.Cu at (60.3, 51.6)
- added U10: 4053, Package_SO:SOIC-16_3.9x9.9mm_P1.27mm, B.Cu at (146.8, 75.4)
- U9: value 74HC4051 -> 74AHCT125; footprint Package_SO:SOIC-16_3.9x9.9mm_P1.27mm -> Package_SO:SOIC-14_3.9x8.7mm_P1.27mm
- moved U9 113.7 mm to (127.0, 38.9), turned to 0 degrees
- moved U1 112.5 mm to (146.8, 34.9)
- moved C49 86.1 mm to (146.8, 81.8), turned to 0 degrees
- moved C50 84.4 mm to (146.8, 65.9), turned to 0 degrees
- moved U8 77.8 mm to (146.8, 89.7)
- moved C41 12.4 mm to (200.0, 84.1)
- moved C42 12.4 mm to (219.1, 84.1)
- moved C19 11.4 mm to (176.2, 24.6), turned to 0 degrees
- moved C22 11.4 mm to (233.4, 23.0), turned to 0 degrees
- moved C28 11.4 mm to (233.4, 42.1), turned to 0 degrees
- moved C40 11.4 mm to (166.7, 86.5)
- moved C23 11.4 mm to (252.4, 32.5), turned to 0 degrees
- moved C24 11.4 mm to (271.5, 37.3), turned to 0 degrees
- moved C27 11.4 mm to (214.3, 37.3), turned to 0 degrees
- moved C30 11.4 mm to (271.5, 56.4), turned to 0 degrees
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Connections:
- U1 pad 1: unconnected-(U1-TX-Pad1) -> LED
- U1 pad 10: SEL10 -> SELX
- U1 pad 11: SEL11 -> SELY
- U1 pad 12: SEL12 -> SELZ
- U1 pad 17: VAL -> VALX
- U1 pad 18: unconnected-(U1-F6-Pad18) -> VALY
- U1 pad 19: unconnected-(U1-F5-Pad19) -> VALZ
- U1 pad 20: unconnected-(U1-F4-Pad20) -> VAL6
- U1 pad 24: unconnected-(U1-RAW-Pad24) -> +5V
- U1 pad 7: SEL00 -> SEL0
- U1 pad 8: SEL01 -> SEL1
- U1 pad 9: SEL02 -> SEL2
- U2 pad 10: SEL11 -> SEL1
- U2 pad 11: SEL10 -> SEL0
- U2 pad 9: SEL12 -> SEL2
- U3 pad 10: SEL11 -> SEL1
- U3 pad 11: SEL10 -> SEL0
- U3 pad 9: SEL12 -> SEL2
- U4 pad 10: SEL11 -> SEL1
- U4 pad 11: SEL10 -> SEL0
- U4 pad 9: SEL12 -> SEL2
- U5 pad 10: SEL11 -> SEL1
- U5 pad 11: SEL10 -> SEL0
- U5 pad 9: SEL12 -> SEL2
- U6 pad 10: SEL11 -> SEL1
- U6 pad 11: SEL10 -> SEL0
- U6 pad 9: SEL12 -> SEL2
- U7 pad 10: SEL11 -> SEL1
- U7 pad 11: SEL10 -> SEL0
- U7 pad 9: SEL12 -> SEL2
- U8 pad 10: SEL11 -> SEL1
- U8 pad 11: SEL10 -> SEL0
- U8 pad 9: SEL12 -> SEL2
- U9 pad 1: VAL4 -> GND
- U9 pad 10: SEL01 -> GND
- U9 pad 11: SEL00 -> GND
- U9 pad 12: VAL3 -> GND
- U9 pad 13: VAL0 -> GND
- U9 pad 14: VAL1 -> +5V
- U9 pad 2: VAL6 -> LED
- U9 pad 3: VAL -> 5VLED
- U9 pad 5: VAL5 -> GND
- U9 pad 9: SEL02 -> GND
Other:
- board outline added: 4.1 x 3.6 mm

Commit message: Update TrueStrike42.kicad_pcb
Rotate left/right hand clusters
Parts:
- moved C49 15.8 mm to (158.8, 71.4)
- moved U8 14.8 mm to (158.8, 81.0)
- moved C6 13.1 mm to (127.7, 32.7), turned to -10 degrees
- moved C1 12.8 mm to (31.7, 28.7), turned to -10 degrees
- moved S6 12.4 mm to (126.9, 37.4), turned to -10 degrees
- moved S1 12.2 mm to (30.9, 33.4), turned to -10 degrees
- moved C74 12.2 mm to (226.4, 94.1), turned to 180 degrees
- moved U9 12.2 mm to (134.6, 48.5)
- moved C4 12.0 mm to (91.3, 19.9), turned to -10 degrees
- moved D6 11.7 mm to (30.1, 38.1), turned to 170 degrees
- moved D1 11.7 mm to (126.1, 42.1), turned to 170 degrees
- moved C5 11.6 mm to (109.0, 29.4), turned to -10 degrees
- moved C72 11.6 mm to (178.2, 101.9), turned to -160 degrees
- moved C3 11.5 mm to (71.7, 21.3), turned to -10 degrees
- moved C43 11.5 mm to (117.5, 35.8), turned to -10 degrees
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Other:
- board size 4.1 x 3.6 mm -> 270.5 x 101.1 mm

Commit message: Update TrueStrike42.kicad_pcb
Finalize board silhouette
Parts:
- U1: moved to B.Cu
- moved U9 40.9 mm to (126.7, 88.6)
- moved C93 40.9 mm to (127.0, 96.3)
- moved C49 38.0 mm to (142.1, 105.6)
- moved U8 38.0 mm to (142.1, 115.1)
- moved C50 16.2 mm to (142.1, 82.6)
- moved U10 16.2 mm to (142.1, 92.1)
- moved C71 15.7 mm to (119.8, 116.7), turned to 150 degrees
- moved D21 14.6 mm to (114.1, 112.5), turned to 150 degrees
- moved S39 14.2 mm to (116.5, 108.4), turned to 150 degrees
- moved C39 13.9 mm to (118.8, 104.3), turned to 150 degrees
- moved C80 12.0 mm to (167.1, 88.8), turned to -75 degrees
- moved C70 11.8 mm to (93.7, 102.6), turned to 165 degrees
- moved D20 11.4 mm to (87.1, 100.0), turned to 165 degrees
- moved D13 11.3 mm to (110.5, 86.6), turned to 165 degrees
- moved C37 11.3 mm to (67.0, 87.8)
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Other:
- board size 270.5 x 101.1 mm -> 273.9 x 109 mm

Commit message: Update TrueStrike42.kicad_pcb
Tracing work in progress
Parts:
- removed the C52 at (43.4, 42.3)
- removed the C53 at (64.3, 38.0)
- removed the C54 at (83.9, 38.4)
- removed the C55 at (100.7, 49.4)
- removed the C56 at (119.1, 54.4)
- removed the C58 at (38.5, 60.7)
- removed C59, C60, C61, C62, C64, C65, C66, C67, C68, C70, C71, C72, C73, C74, C76, C77, C78, C79, C80, C82, C83, C84, C85, C86, C88, C89, C90, C91, C92: 1uF, Capacitor_SMD:C_0805_2012Metric_Pad1.18x1.45mm_HandSolder
- moved C52 104.9 mm to (122.8, 74.5), turned to -90 degrees
- moved C51 100.0 mm to (122.8, 55.7), turned to -90 degrees
- moved C55 33.9 mm to (268.2, 45.0), turned to 30 degrees
- moved D25 33.5 mm to (265.8, 40.8), turned to -150 degrees
- moved S36 33.2 mm to (263.4, 36.7), turned to 30 degrees
- moved C36 32.9 mm to (261.0, 32.6), turned to 30 degrees
- moved D18 32.8 mm to (20.5, 106.6), turned to 180 degrees
- moved S13 32.5 mm to (20.5, 101.8), turned to 0 degrees
- moved D36 32.4 mm to (256.3, 24.3), turned to -150 degrees
- moved S30 32.3 mm to (253.9, 20.2), turned to 30 degrees
- moved C13 32.2 mm to (20.5, 97.0), turned to -90 degrees
- moved C24 32.2 mm to (242.0, -0.40), turned to 30 degrees
- moved C30 32.1 mm to (251.5, 16.1), turned to 30 degrees
- moved S24 32.1 mm to (244.4, 3.73), turned to 30 degrees
- moved C57 32.1 mm to (249.1, 12.0), turned to 30 degrees
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- renumbered C57 to C52, C63 to C53, C69 to C54, C75 to C55, C81 to C56, C87 to C57, C93 to C58
Routing:
- net +3V3: track 0.00 -> 489.4 mm, vias 0 -> 18
- net +5V: track 0.00 -> 465.4 mm, vias 0 -> 18
- net Net-(S1-VOUT): track 0.00 -> 88.2 mm
- net Net-(S7-VOUT): track 0.00 -> 88.1 mm
- net Net-(S13-VOUT): track 0.00 -> 88.1 mm
- net Net-(S8-VOUT): track 0.00 -> 68.4 mm
- net Net-(S2-VOUT): track 0.00 -> 66.9 mm
- net Net-(S14-VOUT): track 0.00 -> 66.9 mm
- net Net-(S15-VOUT): track 0.00 -> 52.6 mm, vias 0 -> 2
- net Net-(S9-VOUT): track 0.00 -> 52.4 mm, vias 0 -> 2
- net Net-(S3-VOUT): track 0.00 -> 52.3 mm, vias 0 -> 2
- net Net-(S16-VOUT): track 0.00 -> 41.8 mm, vias 0 -> 4
- net Net-(S10-VOUT): track 0.00 -> 41.7 mm, vias 0 -> 4
- net Net-(S4-VOUT): track 0.00 -> 41.1 mm, vias 0 -> 4
- net Net-(D6-DOUT): track 0.00 -> 26.0 mm, vias 0 -> 2
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Other:
- board size 273.9 x 109 mm -> 264.7 x 136.6 mm

Commit message: Update TrueStrike42.kicad_pcb
Wiring wip: right side done
Parts:
- moved C55 118.0 mm to (160.9, 94.1), turned to -90 degrees
- moved C57 98.7 mm to (160.9, 56.1), turned to -90 degrees
- moved D25 66.4 mm to (263.2, 107.2), turned to 180 degrees
- moved C36 66.0 mm to (258.1, 98.6), turned to -90 degrees
- moved S36 65.7 mm to (263.2, 102.4), turned to 0 degrees
- moved D18 65.2 mm to (17.9, 41.5), turned to 150 degrees
- moved S13 64.5 mm to (20.3, 37.3), turned to -30 degrees
- moved D36 64.2 mm to (263.2, 88.1), turned to 180 degrees
- moved C30 64.1 mm to (258.1, 79.9), turned to -90 degrees
- moved C13 63.9 mm to (22.7, 33.2), turned to -120 degrees
- moved S30 63.8 mm to (263.2, 83.4), turned to 0 degrees
- moved S24 63.4 mm to (263.2, 64.3), turned to 0 degrees
- moved D37 63.4 mm to (263.2, 69.1), turned to 180 degrees
- moved D7 62.9 mm to (27.4, 25.0), turned to 150 degrees
- moved C24 62.7 mm to (258.2, 60.2), turned to -90 degrees
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Routing:
- net +3V3: track 489.4 -> 977.3 mm, vias 18 -> 51
- net +5V: track 465.4 -> 947.4 mm, vias 18 -> 50
- net Net-(S36-VOUT): track 0.00 -> 89.9 mm, vias 0 -> 2
- net Net-(S24-VOUT): track 0.00 -> 89.2 mm
- net Net-(S30-VOUT): track 0.00 -> 87.6 mm
- net Net-(S29-VOUT): track 0.00 -> 70.7 mm, vias 0 -> 2
- net Net-(S35-VOUT): track 0.00 -> 68.9 mm, vias 0 -> 2
- net Net-(S23-VOUT): track 0.00 -> 67.8 mm
- net Net-(S22-VOUT): track 0.00 -> 62.3 mm, vias 0 -> 2
- net Net-(S34-VOUT): track 0.00 -> 58.3 mm, vias 0 -> 2
- net Net-(S28-VOUT): track 0.00 -> 57.6 mm, vias 0 -> 2
- net Net-(S21-VOUT): track 0.00 -> 42.9 mm, vias 0 -> 2
- net Net-(S33-VOUT): track 0.00 -> 42.7 mm, vias 0 -> 2
- net Net-(S27-VOUT): track 0.00 -> 42.2 mm, vias 0 -> 4
- net Net-(D34-DOUT): track 0.00 -> 23.6 mm, vias 0 -> 2
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Other:
- outline, holes or cut-outs redrawn

Commit message: Update TrueStrike42.kicad_pcb
Wiring finished except for GND
Parts:
- moved C54 72.4 mm to (124.2, 126.1), turned to 60 degrees
- moved C13 43.3 mm to (28.3, 76.1), turned to -105 degrees
- moved D18 41.9 mm to (21.1, 83.2), turned to 165 degrees
- moved S13 41.3 mm to (22.3, 78.6), turned to -15 degrees
- moved C7 41.0 mm to (33.2, 57.7), turned to -105 degrees
- moved D7 39.9 mm to (26.0, 64.8), turned to 165 degrees
- moved S7 39.5 mm to (27.3, 60.2), turned to -15 degrees
- moved C1 39.4 mm to (38.1, 39.3), turned to -105 degrees
- moved C14 38.5 mm to (47.8, 76.6), turned to -105 degrees
- moved D6 38.4 mm to (31.0, 46.4), turned to 165 degrees
- moved S1 38.2 mm to (32.2, 41.8), turned to -15 degrees
- moved D17 36.9 mm to (40.7, 83.6), turned to 165 degrees
- moved S14 36.3 mm to (42.0, 79.0), turned to -15 degrees
- moved C8 36.1 mm to (52.7, 58.2), turned to -105 degrees
- moved D8 34.8 mm to (45.7, 65.2), turned to 165 degrees
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Routing:
- net SEL1: track 0.00 -> 285.1 mm, vias 0 -> 8
- net SEL2: track 0.00 -> 284.4 mm, vias 0 -> 8
- net SEL0: track 0.00 -> 284.1 mm, vias 0 -> 8
- net +5V: track 947.4 -> 1186.0 mm, vias 50 -> 47
- net +3V3: track 977.3 -> 1168.2 mm, vias 51 -> 56
- net Net-(S37-VOUT): track 0.00 -> 80.1 mm
- net Net-(S42-VOUT): track 0.00 -> 78.9 mm
- net VAL6: track 0.00 -> 73.5 mm, vias 0 -> 2
- net VAL2: track 0.00 -> 70.4 mm, vias 0 -> 2
- net Net-(D24-DOUT): track 0.00 -> 69.5 mm, vias 0 -> 2
- net VAL5: track 0.00 -> 64.6 mm, vias 0 -> 4
- net Net-(D18-DOUT): track 0.00 -> 64.3 mm, vias 0 -> 2
- net VAL0: track 0.00 -> 63.6 mm, vias 0 -> 4
- net Net-(S41-VOUT): track 0.00 -> 62.6 mm, vias 0 -> 2
- net Net-(S38-VOUT): track 0.00 -> 58.5 mm
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Other:
- board size 264.7 x 136.6 mm -> 273.9 x 109 mm

Commit message: Update TrueStrike42.kicad_pcb
Finished routing
Parts:
- moved D11 2.07 mm to (104.9, 72.8)
- moved D14 2.07 mm to (100.0, 91.2)
- moved C54 2.07 mm to (126.2, 126.5)
- moved D34 2.07 mm to (231.6, 61.4)
- moved S4 2.07 mm to (94.3, 38.7)
- moved U3 2.07 mm to (112.9, 79.8)
- moved C11 2.07 mm to (110.7, 65.4)
- moved C10 2.07 mm to (95.3, 54.7)
- moved C19 2.07 mm to (164.8, 52.3)
- moved C49 2.07 mm to (146.5, 116.8)
- moved D41 2.07 mm to (190.3, 54.4)
- moved C50 2.07 mm to (153.2, 81.5)
- moved D10 2.07 mm to (88.2, 61.7)
- moved D23 2.07 mm to (205.1, 109.6)
- moved D6 2.07 mm to (33.0, 46.9)
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Routing:
- net SELY: track 16.7 -> 18.1 mm
- net SELZ: track 15.3 -> 16.3 mm
- net Net-(D24-DOUT): track 69.5 -> 68.7 mm
Other:
- outline, holes or cut-outs redrawn
