File: hw/pcb/TrueStrike42.kicad_pcb (KiCad board)
At the start: 2 copper layers, 273.9 x 109 mm, 152 parts, among them U1 ProMicro, U10 4053, U2 74HC4051, U3 74HC4051, U4 74HC4051, U5 74HC4051, U6 74HC4051, U7 74HC4051, U8 74HC4051, U9 74AHCT125

Commit message: Add LED screen and a reset switch
Parts:
- added Brd1: SSD1306, SSD1306:128x64OLED, F.Cu at (150.0, 95.6)
- added SW1: SW_Push, Button_Switch_SMD:SW_Tactile_SPST_NO_Straight_CK_PTS636Sx25SMTRLFS, B.Cu at (150.1, 97.8)
Connections:
- U1 pad 5: unconnected-(U1-SDA-Pad5) -> SDA
- U1 pad 6: unconnected-(U1-SCL-Pad6) -> SCL
Routing:
- net RESET: track 0.00 -> 57.1 mm, vias 0 -> 4
- net SDA: track 0.00 -> 56.8 mm, vias 0 -> 3
- net SCL: track 0.00 -> 51.4 mm, vias 0 -> 3
- net +3V3: track 1168.2 -> 1166.5 mm

Commit message: GND fill + DRC check pass
Parts:
- moved C57 4.80 mm to (166.5, 65.4)
- moved S9 4.80 mm to (71.3, 61.3)
- moved D29 4.80 mm to (201.6, 95.7)
- moved S16 4.80 mm to (86.0, 80.1)
- moved D19 4.80 mm to (76.4, 111.5)
- moved U4 4.80 mm to (109.4, 102.8)
- moved C38 4.80 mm to (102.5, 106.8)
- moved C4 4.80 mm to (101.7, 40.7)
- moved C26 4.80 mm to (192.1, 69.7)
- moved D26 4.80 mm to (258.9, 88.6)
- moved C12 4.80 mm to (131.9, 75.2)
- moved C11 4.80 mm to (112.2, 69.9)
- moved C40 4.80 mm to (179.6, 116.6)
- moved D21 4.80 mm to (123.5, 126.6)
- moved S14 4.80 mm to (45.5, 84.0)
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Routing:
- net GND: track 0.00 -> 23.4 mm, vias 0 -> 44
- net Net-(D24-DOUT): track 68.7 -> 70.2 mm
- net 5VLED: track 33.9 -> 35.2 mm
- net Net-(S3-VOUT): track 52.3 -> 53.3 mm
- net Net-(S33-VOUT): track 43.4 -> 44.2 mm
- net Net-(S24-VOUT): track 91.8 -> 92.5 mm
- net Net-(S37-VOUT): track 80.1 -> 80.8 mm
- net Net-(S14-VOUT): track 68.0 -> 67.3 mm
- net Net-(S15-VOUT): track 52.6 -> 53.2 mm
- net Net-(S2-VOUT): track 68.1 -> 68.6 mm
- net Net-(S42-VOUT): track 78.9 -> 79.4 mm
- added copper zone on B.Cu, net GND
- added copper zone on F.Cu, net GND
Other:
- outline, holes or cut-outs redrawn

Commit message: Update functional silkscreens
Parts:
- moved C54 4.54 mm to (126.2, 126.8)
- moved D34 4.54 mm to (231.6, 61.6)
- moved S7 4.54 mm to (29.3, 61.0)
- moved S8 4.54 mm to (48.9, 61.3)
- moved U2 4.54 mm to (117.8, 61.7)
- moved C11 4.54 mm to (110.7, 65.6)
- moved C12 4.54 mm to (130.4, 70.9)
- moved C19 4.54 mm to (164.8, 52.6)
- moved C20 4.54 mm to (183.2, 47.6)
- moved C24 4.54 mm to (260.0, 39.9)
- moved C26 4.54 mm to (190.6, 65.4)
- moved C27 4.54 mm to (204.9, 55.2)
- moved C29 4.54 mm to (245.4, 59.1)
- moved C30 4.54 mm to (265.0, 58.9)
- moved C31 4.54 mm to (174.5, 89.4)
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- renumbered SW1 to RESET
Other:
- board text added: "12/B6"
- board text added: "13/B2"
- board text added: "14/B3"
- board text added: "15/B1"
- board text added: "3V3"
- board text added: "5V"
- board text added: "A0/F7"
- board text added: "A1/F6"
- board text added: "A2/F5"
- board text added: "A3/F4"
- board text added: "B4/8"
- board text added: "B5/9"
- board text added: "C6/5"
- board text added: "D2/RX"
- board text added: "D3/TX"
- board text added: "D4/4"
- board text added: "D7/6"
- board text added: "E6/7"
- board text added: "GND"
- board text added: "RESET"
- board text added: "SCL"
- board text added: "SDA"
