File: hw/pcb/TrueStrike42.kicad_pcb (KiCad board)
At the start: 2 copper layers, 273.9 x 109 mm, 154 parts, among them U1 ProMicro, U10 4053, U2 74HC4051, U3 74HC4051, U4 74HC4051, U5 74HC4051, U6 74HC4051, U7 74HC4051, U8 74HC4051, U9 74AHCT125

Commit message: Update TrueStrike42.kicad_pcb
Add mounting holes
Parts:
- added REF**: MountingHole_3.5mm, MountingHole:MountingHole_3.5mm, F.Cu at (269.5, 93.7)
- added REF**: MountingHole_2.2mm_M2, MountingHole:MountingHole_2.2mm_M2, F.Cu at (142.6, 79.7)
- added REF**: MountingHole_2.2mm_M2, MountingHole:MountingHole_2.2mm_M2, F.Cu at (171.8, 108.2)
- added REF**: MountingHole_3.5mm, MountingHole:MountingHole_3.5mm, F.Cu at (48.9, 35.4)
- added REF**: MountingHole_2.2mm_M2, MountingHole:MountingHole_2.2mm_M2, F.Cu at (166.5, 79.7)
- added REF**: MountingHole_2.2mm_M2, MountingHole:MountingHole_2.2mm_M2, F.Cu at (136.6, 108.2)
- added REF**: MountingHole_3.5mm, MountingHole:MountingHole_3.5mm, F.Cu at (39.7, 93.6)
- added REF**: MountingHole_3.5mm, MountingHole:MountingHole_3.5mm, F.Cu at (260.3, 35.5)
- added REF**: MountingHole_3.5mm, MountingHole:MountingHole_3.5mm, F.Cu at (111.6, 39.0)
- added REF**: MountingHole_3.5mm, MountingHole:MountingHole_3.5mm, F.Cu at (197.6, 39.1)
- added REF**: MountingHole_3.5mm, MountingHole:MountingHole_3.5mm, F.Cu at (111.3, 109.7)
- added REF**: MountingHole_3.5mm, MountingHole:MountingHole_3.5mm, F.Cu at (197.9, 109.8)
- moved C31 5.08 mm to (179.1, 91.6)
- moved S21 5.08 mm to (210.4, 41.2)
- moved U9 5.08 mm to (144.5, 88.3)
- moved S12 5.08 mm to (129.1, 75.6)
- moved D5 5.08 mm to (57.2, 49.7)
- moved S16 5.08 mm to (89.0, 78.0)
- moved D14 5.08 mm to (104.6, 93.6)
- moved C46 5.08 mm to (184.4, 54.7)
- moved D34 5.08 mm to (236.2, 63.9)
- moved S42 5.08 mm to (229.7, 104.6)
- moved C7 5.08 mm to (39.8, 60.7)
- moved D32 5.08 mm to (199.8, 75.2)
- moved D9 5.08 mm to (73.1, 63.9)
- moved U4 5.08 mm to (112.5, 100.7)
- moved C32 5.08 mm to (200.0, 86.0)
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Routing:
- net Net-(D24-DOUT): track 70.2 -> 70.9 mm
- net Net-(D18-DOUT): track 64.7 -> 65.4 mm
- net +5V: track 1185.9 -> 1186.6 mm

Commit message: Add logo, fixed wrong pinouts for sensors
Parts:
- added G***: LOGO, project-specific-library:True-Strike-icon, B.Cu at (241.4, 93.3)
- moved S4 6.78 mm to (92.7, 43.9)
- moved REF** 6.78 mm to (160.3, 82.4)
- moved C8 6.78 mm to (53.1, 63.8)
- moved S13 6.78 mm to (22.7, 84.3)
- moved REF** 6.78 mm to (165.6, 110.9)
- moved C20 6.78 mm to (181.6, 52.5)
- moved C5 6.78 mm to (115.3, 52.6)
- moved S3 6.78 mm to (73.0, 43.5)
- moved D39 6.78 mm to (225.0, 48.1)
- moved D23 6.78 mm to (203.4, 114.7)
- moved C46 6.78 mm to (178.2, 57.4)
- moved S38 6.78 mm to (94.6, 110.1)
- moved C13 6.78 mm to (28.6, 81.8)
- moved U7 6.78 mm to (190.5, 103.4)
- moved C27 6.78 mm to (203.3, 60.0)
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- renumbered RESET to SW1
Connections:
- S1 pad 2: GND -> Net-(S1-GND)
- S1 pad 3: Net-(S1-VOUT) -> GND
- S10 pad 2: GND -> Net-(S10-GND)
- S10 pad 3: Net-(S10-VOUT) -> GND
- S11 pad 2: GND -> Net-(S11-GND)
- S11 pad 3: Net-(S11-VOUT) -> GND
- S12 pad 2: GND -> Net-(S12-GND)
- S12 pad 3: Net-(S12-VOUT) -> GND
- S13 pad 2: GND -> Net-(S13-GND)
- S13 pad 3: Net-(S13-VOUT) -> GND
- S14 pad 2: GND -> Net-(S14-GND)
- S14 pad 3: Net-(S14-VOUT) -> GND
- S15 pad 2: GND -> Net-(S15-GND)
- S15 pad 3: Net-(S15-VOUT) -> GND
- S16 pad 2: GND -> Net-(S16-GND)
- S16 pad 3: Net-(S16-VOUT) -> GND
- S17 pad 2: GND -> Net-(S17-GND)
- S17 pad 3: Net-(S17-VOUT) -> GND
- S18 pad 2: GND -> Net-(S18-GND)
- S18 pad 3: Net-(S18-VOUT) -> GND
- S19 pad 2: GND -> Net-(S19-GND)
- S19 pad 3: Net-(S19-VOUT) -> GND
- S2 pad 2: GND -> Net-(S2-GND)
- S2 pad 3: Net-(S2-VOUT) -> GND
- S20 pad 2: GND -> Net-(S20-GND)
- S20 pad 3: Net-(S20-VOUT) -> GND
- S21 pad 2: GND -> Net-(S21-GND)
- S21 pad 3: Net-(S21-VOUT) -> GND
- S22 pad 2: GND -> Net-(S22-GND)
- S22 pad 3: Net-(S22-VOUT) -> GND
- S23 pad 2: GND -> Net-(S23-GND)
- S23 pad 3: Net-(S23-VOUT) -> GND
- S24 pad 2: GND -> Net-(S24-GND)
- S24 pad 3: Net-(S24-VOUT) -> GND
- S25 pad 2: GND -> Net-(S25-GND)
- S25 pad 3: Net-(S25-VOUT) -> GND
- S26 pad 2: GND -> Net-(S26-GND)
- S26 pad 3: Net-(S26-VOUT) -> GND
- S27 pad 2: GND -> Net-(S27-GND)
- S27 pad 3: Net-(S27-VOUT) -> GND
- S28 pad 2: GND -> Net-(S28-GND)
- S28 pad 3: Net-(S28-VOUT) -> GND
- S29 pad 2: GND -> Net-(S29-GND)
- S29 pad 3: Net-(S29-VOUT) -> GND
- S3 pad 2: GND -> Net-(S3-GND)
- S3 pad 3: Net-(S3-VOUT) -> GND
- S30 pad 2: GND -> Net-(S30-GND)
- S30 pad 3: Net-(S30-VOUT) -> GND
- S31 pad 2: GND -> Net-(S31-GND)
- S31 pad 3: Net-(S31-VOUT) -> GND
- S32 pad 2: GND -> Net-(S32-GND)
- S32 pad 3: Net-(S32-VOUT) -> GND
- S33 pad 2: GND -> Net-(S33-GND)
- S33 pad 3: Net-(S33-VOUT) -> GND
- S34 pad 2: GND -> Net-(S34-GND)
- S34 pad 3: Net-(S34-VOUT) -> GND
- S35 pad 2: GND -> Net-(S35-GND)
- S35 pad 3: Net-(S35-VOUT) -> GND
- S36 pad 2: GND -> Net-(S36-GND)
- S36 pad 3: Net-(S36-VOUT) -> GND
- S37 pad 2: GND -> Net-(S37-GND)
- S37 pad 3: Net-(S37-VOUT) -> GND
- S38 pad 2: GND -> Net-(S38-GND)
- S38 pad 3: Net-(S38-VOUT) -> GND
- S39 pad 2: GND -> Net-(S39-GND)
- S39 pad 3: Net-(S39-VOUT) -> GND
- S4 pad 2: GND -> Net-(S4-GND)
- S4 pad 3: Net-(S4-VOUT) -> GND
- S40 pad 2: GND -> Net-(S40-GND)
- S40 pad 3: Net-(S40-VOUT) -> GND
- S41 pad 2: GND -> Net-(S41-GND)
- S41 pad 3: Net-(S41-VOUT) -> GND
- S42 pad 2: GND -> Net-(S42-GND)
- S42 pad 3: Net-(S42-VOUT) -> GND
- S5 pad 2: GND -> Net-(S5-GND)
- S5 pad 3: Net-(S5-VOUT) -> GND
- S6 pad 2: GND -> Net-(S6-GND)
- S6 pad 3: Net-(S6-VOUT) -> GND
- S7 pad 2: GND -> Net-(S7-GND)
- S7 pad 3: Net-(S7-VOUT) -> GND
- S8 pad 2: GND -> Net-(S8-GND)
- S8 pad 3: Net-(S8-VOUT) -> GND
- S9 pad 2: GND -> Net-(S9-GND)
- S9 pad 3: Net-(S9-VOUT) -> GND
- U2 pad 1: Net-(S5-VOUT) -> Net-(S5-GND)
- U2 pad 12: Net-(S4-VOUT) -> Net-(S4-GND)
- U2 pad 13: Net-(S1-VOUT) -> Net-(S1-GND)
- U2 pad 14: Net-(S2-VOUT) -> Net-(S2-GND)
- U2 pad 15: Net-(S3-VOUT) -> Net-(S3-GND)
- U2 pad 5: Net-(S6-VOUT) -> Net-(S6-GND)
- U3 pad 1: Net-(S11-VOUT) -> Net-(S11-GND)
- U3 pad 12: Net-(S10-VOUT) -> Net-(S10-GND)
- U3 pad 13: Net-(S7-VOUT) -> Net-(S7-GND)
- U3 pad 14: Net-(S8-VOUT) -> Net-(S8-GND)
- U3 pad 15: Net-(S9-VOUT) -> Net-(S9-GND)
- U3 pad 5: Net-(S12-VOUT) -> Net-(S12-GND)
- U4 pad 1: Net-(S17-VOUT) -> Net-(S17-GND)
- U4 pad 12: Net-(S16-VOUT) -> Net-(S16-GND)
- U4 pad 13: Net-(S13-VOUT) -> Net-(S13-GND)
- U4 pad 14: Net-(S14-VOUT) -> Net-(S14-GND)
- U4 pad 15: Net-(S15-VOUT) -> Net-(S15-GND)
- U4 pad 5: Net-(S18-VOUT) -> Net-(S18-GND)
- U5 pad 1: Net-(S23-VOUT) -> Net-(S23-GND)
- U5 pad 12: Net-(S22-VOUT) -> Net-(S22-GND)
- U5 pad 13: Net-(S19-VOUT) -> Net-(S19-GND)
- U5 pad 14: Net-(S20-VOUT) -> Net-(S20-GND)
- U5 pad 15: Net-(S21-VOUT) -> Net-(S21-GND)
- U5 pad 5: Net-(S24-VOUT) -> Net-(S24-GND)
- U6 pad 1: Net-(S29-VOUT) -> Net-(S29-GND)
- U6 pad 12: Net-(S28-VOUT) -> Net-(S28-GND)
- U6 pad 13: Net-(S25-VOUT) -> Net-(S25-GND)
- U6 pad 14: Net-(S26-VOUT) -> Net-(S26-GND)
- U6 pad 15: Net-(S27-VOUT) -> Net-(S27-GND)
- U6 pad 5: Net-(S30-VOUT) -> Net-(S30-GND)
- U7 pad 1: Net-(S35-VOUT) -> Net-(S35-GND)
- U7 pad 12: Net-(S34-VOUT) -> Net-(S34-GND)
- U7 pad 13: Net-(S31-VOUT) -> Net-(S31-GND)
- U7 pad 14: Net-(S32-VOUT) -> Net-(S32-GND)
- U7 pad 15: Net-(S33-VOUT) -> Net-(S33-GND)
- U7 pad 5: Net-(S36-VOUT) -> Net-(S36-GND)
- U8 pad 1: Net-(S41-VOUT) -> Net-(S41-GND)
- U8 pad 12: Net-(S40-VOUT) -> Net-(S40-GND)
- U8 pad 13: Net-(S37-VOUT) -> Net-(S37-GND)
- U8 pad 14: Net-(S38-VOUT) -> Net-(S38-GND)
- U8 pad 15: Net-(S39-VOUT) -> Net-(S39-GND)
- U8 pad 5: Net-(S42-VOUT) -> Net-(S42-GND)
Routing:
- net Net-(S24-GND): track 0.00 -> 94.0 mm, vias 0 -> 2
- net Net-(S24-VOUT): track 92.5 -> 0.00 mm, vias 2 -> 0
- net Net-(S36-GND): track 0.00 -> 91.5 mm, vias 0 -> 2
- net Net-(S30-GND): track 0.00 -> 90.4 mm
- net Net-(S36-VOUT): track 90.0 -> 0.00 mm, vias 2 -> 0
- net Net-(S7-VOUT): track 88.1 -> 0.00 mm
- net Net-(S1-VOUT): track 88.0 -> 0.00 mm
- net Net-(S13-VOUT): track 87.9 -> 0.00 mm
- net Net-(S30-VOUT): track 87.6 -> 0.00 mm
- net Net-(S7-GND): track 0.00 -> 86.7 mm
- net Net-(S1-GND): track 0.00 -> 86.5 mm
- net Net-(S13-GND): track 0.00 -> 86.4 mm
- net Net-(S42-GND): track 0.00 -> 80.8 mm
- net Net-(S37-VOUT): track 80.8 -> 0.00 mm
- net Net-(S42-VOUT): track 79.4 -> 0.00 mm
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Other:
- outline, holes or cut-outs redrawn
- board text added: "Rev.1"
- board text added: "TrueStrike42"

Commit message: Update reset button label
Parts:
- renumbered SW1 to RESET
Changed lines of the file:
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@@
 		(descr "Tactile switch, SPST, 6.0x3.5 mm, H2.5 mm, straight, NO, gull wing leads: https://www.ckswitches.com/media/2779/pts636.pdf")
 		(tags "switch tactile SPST 1P1T straight NO SMTR C&K")
-		(property "Reference" "SW1"
+		(property "Reference" "RESET"
 			(at 0 3 0)
 			(unlocked yes)

Commit message: Add order number locator for JLCPCB
Other:
- board text added: "JLCJLCJLCJLC"
Changed lines of the file:
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@@
+		)
+	)
+	(gr_text "JLCJLCJLCJLC"
+		(at 148.4 139.5 0)
+		(layer "B.SilkS")
+		(effects
+			(font
+				(size 0.8 0.8)
+				(thickness 0.1)
+			)
+			(justify bottom mirror)
 		)
 	)
