File: hw/pcb/TrueStrike42.kicad_sch (KiCad schematic)
At the start: 102 parts, among them U1 74HC4051, U10 74HC4051, U2 74HC4051, U3 74HC4051, U4 74HC4051, U5 74HC4051, U6 Teensy4.1, U7 ProMicro, U8 74HC4051, U9 74HC4051

Commit message: Update TrueStrike42.kicad_sch
Parts:
- removed U6: Teensy4.1, symbol teensy:Teensy4.1
- C1, C2, C3, C4, C49, C5, C50, C6: footprint (none) -> Capacitor_SMD:C_0805_2012Metric_Pad1.18x1.45mm_HandSolder
- C10: renamed from C13; footprint (none) -> Capacitor_SMD:C_0805_2012Metric_Pad1.18x1.45mm_HandSolder
- C11: renamed from C14; footprint (none) -> Capacitor_SMD:C_0805_2012Metric_Pad1.18x1.45mm_HandSolder
- C12: renamed from C15; footprint (none) -> Capacitor_SMD:C_0805_2012Metric_Pad1.18x1.45mm_HandSolder
- C13: renamed from C7; footprint (none) -> Capacitor_SMD:C_0805_2012Metric_Pad1.18x1.45mm_HandSolder
- C14: renamed from C8; footprint (none) -> Capacitor_SMD:C_0805_2012Metric_Pad1.18x1.45mm_HandSolder
- C15: renamed from C16; footprint (none) -> Capacitor_SMD:C_0805_2012Metric_Pad1.18x1.45mm_HandSolder
- C16: renamed from C17; footprint (none) -> Capacitor_SMD:C_0805_2012Metric_Pad1.18x1.45mm_HandSolder
- C17: renamed from C19; footprint (none) -> Capacitor_SMD:C_0805_2012Metric_Pad1.18x1.45mm_HandSolder
- C18: renamed from C20; footprint (none) -> Capacitor_SMD:C_0805_2012Metric_Pad1.18x1.45mm_HandSolder
- C19: renamed from C22; footprint (none) -> Capacitor_SMD:C_0805_2012Metric_Pad1.18x1.45mm_HandSolder
- C20: renamed from C23; footprint (none) -> Capacitor_SMD:C_0805_2012Metric_Pad1.18x1.45mm_HandSolder
- C21: renamed from C24; footprint (none) -> Capacitor_SMD:C_0805_2012Metric_Pad1.18x1.45mm_HandSolder
- C22: renamed from C25; footprint (none) -> Capacitor_SMD:C_0805_2012Metric_Pad1.18x1.45mm_HandSolder
- C23: renamed from C26; footprint (none) -> Capacitor_SMD:C_0805_2012Metric_Pad1.18x1.45mm_HandSolder
- C24: renamed from C27; footprint (none) -> Capacitor_SMD:C_0805_2012Metric_Pad1.18x1.45mm_HandSolder
- C25: renamed from C29; footprint (none) -> Capacitor_SMD:C_0805_2012Metric_Pad1.18x1.45mm_HandSolder
- C26: renamed from C30; footprint (none) -> Capacitor_SMD:C_0805_2012Metric_Pad1.18x1.45mm_HandSolder
- C27: renamed from C31; footprint (none) -> Capacitor_SMD:C_0805_2012Metric_Pad1.18x1.45mm_HandSolder
- C28: renamed from C32; footprint (none) -> Capacitor_SMD:C_0805_2012Metric_Pad1.18x1.45mm_HandSolder
- C29: renamed from C33; footprint (none) -> Capacitor_SMD:C_0805_2012Metric_Pad1.18x1.45mm_HandSolder
- C30: renamed from C34; footprint (none) -> Capacitor_SMD:C_0805_2012Metric_Pad1.18x1.45mm_HandSolder
- C31: renamed from C36; footprint (none) -> Capacitor_SMD:C_0805_2012Metric_Pad1.18x1.45mm_HandSolder
- C32: renamed from C37; footprint (none) -> Capacitor_SMD:C_0805_2012Metric_Pad1.18x1.45mm_HandSolder
- C33: renamed from C38; footprint (none) -> Capacitor_SMD:C_0805_2012Metric_Pad1.18x1.45mm_HandSolder
- C34: renamed from C39; footprint (none) -> Capacitor_SMD:C_0805_2012Metric_Pad1.18x1.45mm_HandSolder
- C35: renamed from C40; footprint (none) -> Capacitor_SMD:C_0805_2012Metric_Pad1.18x1.45mm_HandSolder
- C36: renamed from C41; footprint (none) -> Capacitor_SMD:C_0805_2012Metric_Pad1.18x1.45mm_HandSolder
- C37: renamed from C43; footprint (none) -> Capacitor_SMD:C_0805_2012Metric_Pad1.18x1.45mm_HandSolder
- C38: renamed from C44; footprint (none) -> Capacitor_SMD:C_0805_2012Metric_Pad1.18x1.45mm_HandSolder
- C39: renamed from C45; footprint (none) -> Capacitor_SMD:C_0805_2012Metric_Pad1.18x1.45mm_HandSolder
- C40: renamed from C46; footprint (none) -> Capacitor_SMD:C_0805_2012Metric_Pad1.18x1.45mm_HandSolder
- C41: renamed from C47; footprint (none) -> Capacitor_SMD:C_0805_2012Metric_Pad1.18x1.45mm_HandSolder
- C42: renamed from C48; footprint (none) -> Capacitor_SMD:C_0805_2012Metric_Pad1.18x1.45mm_HandSolder
- C43: renamed from C9; footprint (none) -> Capacitor_SMD:C_0805_2012Metric_Pad1.18x1.45mm_HandSolder
- C44: renamed from C18; footprint (none) -> Capacitor_SMD:C_0805_2012Metric_Pad1.18x1.45mm_HandSolder
- C45: renamed from C21; footprint (none) -> Capacitor_SMD:C_0805_2012Metric_Pad1.18x1.45mm_HandSolder
- C46: renamed from C28; footprint (none) -> Capacitor_SMD:C_0805_2012Metric_Pad1.18x1.45mm_HandSolder
- C47: renamed from C35; footprint (none) -> Capacitor_SMD:C_0805_2012Metric_Pad1.18x1.45mm_HandSolder
- C48: renamed from C42; footprint (none) -> Capacitor_SMD:C_0805_2012Metric_Pad1.18x1.45mm_HandSolder
- C7: renamed from C10; footprint (none) -> Capacitor_SMD:C_0805_2012Metric_Pad1.18x1.45mm_HandSolder
- C8: renamed from C11; footprint (none) -> Capacitor_SMD:C_0805_2012Metric_Pad1.18x1.45mm_HandSolder
- C9: renamed from C12; footprint (none) -> Capacitor_SMD:C_0805_2012Metric_Pad1.18x1.45mm_HandSolder
- S1, S15, S16, S17, S18, S19, S2, S20, S21, S22, S23, S24, S25, S26, S27, S28, S29, S3, S30, S31, S32, S33, S34, S35, S36, S37, S38, S4, S41, S42, S5, S6: footprint (none) -> project-specific-library:HE-Switch-1U
- S10: renamed from S12; footprint (none) -> project-specific-library:HE-Switch-1U
- S11: renamed from S13; footprint (none) -> project-specific-library:HE-Switch-1U
- S12: renamed from S14; footprint (none) -> project-specific-library:HE-Switch-1U
- S13: renamed from S7; footprint (none) -> project-specific-library:HE-Switch-1U
- S14: renamed from S8; footprint (none) -> project-specific-library:HE-Switch-1U
- S39, S40: footprint (none) -> project-specific-library:HE-Switch-2U
- S7: renamed from S9; footprint (none) -> project-specific-library:HE-Switch-1U
- S8: renamed from S10; footprint (none) -> project-specific-library:HE-Switch-1U
- S9: renamed from S11; footprint (none) -> project-specific-library:HE-Switch-1U
- U1: renamed from U7; footprint (none) -> promicro:ProMicro
- U2: renamed from U1; footprint (none) -> Package_SO:SOIC-16_3.9x9.9mm_P1.27mm
- U3: renamed from U2; footprint (none) -> Package_SO:SOIC-16_3.9x9.9mm_P1.27mm
- U4: renamed from U3; footprint (none) -> Package_SO:SOIC-16_3.9x9.9mm_P1.27mm
- U5: renamed from U4; footprint (none) -> Package_SO:SOIC-16_3.9x9.9mm_P1.27mm
- U6: renamed from U5; footprint (none) -> Package_SO:SOIC-16_3.9x9.9mm_P1.27mm
- U7: renamed from U8; footprint (none) -> Package_SO:SOIC-16_3.9x9.9mm_P1.27mm
- U8: renamed from U9; footprint (none) -> Package_SO:SOIC-16_3.9x9.9mm_P1.27mm
- U9: renamed from U10; footprint (none) -> Package_SO:SOIC-16_3.9x9.9mm_P1.27mm
Other:
- moved on the sheet: C50, U9

Commit message: Update TrueStrike42.kicad_sch
Add LED matrix schematics
Parts:
- removed U9: 74HC4051, Package_SO:SOIC-16_3.9x9.9mm_P1.27mm, symbol 74xx:74HC4051
- added C51, C52, C53, C54, C55, C56, C57, C58, C59, C60, C61, C62, C63, C64, C65, C66, C67, C68, C69, C70, C71, C72, C73, C74, C75, C76, C77, C78, C79, C80, C81, C82, C83, C84, C85, C86, C87, C88, C89, C90, C91, C92, C93: 1uF, Capacitor_SMD:C_0805_2012Metric_Pad1.18x1.45mm_HandSolder, symbol Device:C_Small
- added D1, D10, D11, D12, D13, D14, D15, D16, D17, D18, D19, D2, D20, D21, D22, D23, D24, D25, D26, D27, D28, D29, D3, D30, D31, D32, D33, D34, D35, D36, D37, D38, D39, D4, D40, D41, D42, D5, D6, D7, D8, D9: SK6812MINI-E, SkeletonKBD-Parts:SK6812MINI-E_nusumi, symbol SkeletonKBD-Parts:SK6812MINI-E
- added U10: 4053, Package_SO:SOIC-16_3.9x9.9mm_P1.27mm, symbol 4xxx:4053
- added U9: 74AHCT125, Package_SO:SOIC-14_3.9x8.7mm_P1.27mm, symbol 74xx:74AHCT125
- S39, S40: footprint project-specific-library:HE-Switch-2U -> project-specific-library:HE-Switch-2U_V
Connections:
- net +3V3: now also U10.16 (VDD)
- net GND: now also C51.2, C52.2, C53.2, C54.2, C55.2, C56.2, C57.1, C58.1, C59.1, C60.1, C61.1, C62.1, C63.2, C64.2, C65.2, C66.2, C67.2, C68.2, C69.1, C70.1, C71.1, C72.1, C73.1, C74.1, C75.2, C76.2, C77.2, C78.2, C79.2, C80.2, C81.1, C82.1, C83.1, C84.1, C85.1, C86.1, C87.2, C88.2, C89.2, C90.2, C91.2, C92.2, C93.2, D1.3 (VSS), D10.3 (VSS), D11.3 (VSS), D12.3 (VSS), D13.3 (VSS), D14.3 (VSS), D15.3 (VSS), D16.3 (VSS), D17.3 (VSS), D18.3 (VSS), D19.3 (VSS), D2.3 (VSS), D20.3 (VSS), D21.3 (VSS), D22.3 (VSS), D23.3 (VSS), D24.3 (VSS), D25.3 (VSS), D26.3 (VSS), D27.3 (VSS), D28.3 (VSS), D29.3 (VSS), D3.3 (VSS), D30.3 (VSS), D31.3 (VSS), D32.3 (VSS), D33.3 (VSS), D34.3 (VSS), D35.3 (VSS), D36.3 (VSS), D37.3 (VSS), D38.3 (VSS), D39.3 (VSS), D4.3 (VSS), D40.3 (VSS), D41.3 (VSS), D42.3 (VSS), D5.3 (VSS), D6.3 (VSS), D7.3 (VSS), D8.3 (VSS), D9.3 (VSS), U10.6 (Inh), U10.7 (VEE), U10.8 (VSS), U9.1, U9.10, U9.11, U9.12, U9.13, U9.4, U9.5, U9.6, U9.7 (GND), U9.8, U9.9
- net VAL0: now also U10.12 (X0)
- net VAL1: now also U10.13 (X1)
- net VAL2: now also U10.2 (Y0)
- net VAL3: now also U10.1 (Y1)
- net VAL4: now also U10.5 (Z0)
- net VAL5: now also U10.3 (Z1)
- net VAL6: now also U1.20 (F4)
- net LED: now reaches U1.1 (TX)
- net LED: now also U9.2
- net VALY: now reaches U1.18 (F6)
- net VALY: now also U10.15 (Y)
- net VALZ: now reaches U1.19 (F5)
- net VALZ: now also U10.4 (Z)
- net +5V: now reaches U1.24 (RAW)
- net +5V: now also C51.1, C52.1, C53.1, C54.1, C55.1, C56.1, C57.2, C58.2, C59.2, C60.2, C61.2, C62.2, C63.1, C64.1, C65.1, C66.1, C67.1, C68.1, C69.2, C70.2, C71.2, C72.2, C73.2, C74.2, C75.1, C76.1, C77.1, C78.1, C79.1, C80.1, C81.2, C82.2, C83.2, C84.2, C85.2, C86.2, C87.1, C88.1, C89.1, C90.1, C91.1, C92.1, C93.1, D1.1 (VDD), D10.1 (VDD), D11.1 (VDD), D12.1 (VDD), D13.1 (VDD), D14.1 (VDD), D15.1 (VDD), D16.1 (VDD), D17.1 (VDD), D18.1 (VDD), D19.1 (VDD), D2.1 (VDD), D20.1 (VDD), D21.1 (VDD), D22.1 (VDD), D23.1 (VDD), D24.1 (VDD), D25.1 (VDD), D26.1 (VDD), D27.1 (VDD), D28.1 (VDD), D29.1 (VDD), D3.1 (VDD), D30.1 (VDD), D31.1 (VDD), D32.1 (VDD), D33.1 (VDD), D34.1 (VDD), D35.1 (VDD), D36.1 (VDD), D37.1 (VDD), D38.1 (VDD), D39.1 (VDD), D4.1 (VDD), D40.1 (VDD), D41.1 (VDD), D42.1 (VDD), D5.1 (VDD), D6.1 (VDD), D7.1 (VDD), D8.1 (VDD), D9.1 (VDD), U9.14 (VCC)
- net SEL00 renamed SEL0
- net SEL0: now also U2.11 (S0), U3.11 (S0), U4.11 (S0), U5.11 (S0), U6.11 (S0), U7.11 (S0), U8.11 (S0)
- net SEL01 renamed SEL1
- net SEL1: now also U2.10 (S1), U3.10 (S1), U4.10 (S1), U5.10 (S1), U6.10 (S1), U7.10 (S1), U8.10 (S1)
- net SEL02 renamed SEL2
- net SEL2: now also U2.9 (S2), U3.9 (S2), U4.9 (S2), U5.9 (S2), U6.9 (S2), U7.9 (S2), U8.9 (S2)
- removed net SEL10: U1.10 (E6), U2.11 (S0), U3.11 (S0), U4.11 (S0), U5.11 (S0), U6.11 (S0), U7.11 (S0), U8.11 (S0)
- removed net SEL11: U1.11 (B4), U2.10 (S1), U3.10 (S1), U4.10 (S1), U5.10 (S1), U6.10 (S1), U7.10 (S1), U8.10 (S1)
- removed net SEL12: U1.12 (B5), U2.9 (S2), U3.9 (S2), U4.9 (S2), U5.9 (S2), U6.9 (S2), U7.9 (S2), U8.9 (S2)
- net VAL renamed VALX
- net VALX: now also U10.14 (X)
- new net: D33.2 (DOUT), D34.4 (DIN)
- new net: D32.2 (DOUT), D33.4 (DIN)
- new net: D34.2 (DOUT), D35.4 (DIN)
- new net: D23.2 (DOUT), D24.4 (DIN)
- new net: D22.2 (DOUT), D23.4 (DIN)
- new net: D25.2 (DOUT), D26.4 (DIN)
- new net: D24.2 (DOUT), D25.4 (DIN)
- new net: D21.2 (DOUT), D22.4 (DIN)
- new net: D3.2 (DOUT), D4.4 (DIN)
- new net: D2.2 (DOUT), D3.4 (DIN)
- new net: D20.2 (DOUT), D21.4 (DIN)
- new net: D19.2 (DOUT), D20.4 (DIN)
- new net: D28.2 (DOUT), D29.4 (DIN)
- new net: D27.2 (DOUT), D28.4 (DIN)
- new net: D15.2 (DOUT), D16.4 (DIN)
- new net: D14.2 (DOUT), D15.4 (DIN)
- new net: D26.2 (DOUT), D27.4 (DIN)
- new net: D40.2 (DOUT), D41.4 (DIN)
- new net: D39.2 (DOUT), D40.4 (DIN)
- new net: D7.2 (DOUT), D8.4 (DIN)
- new net: D6.2 (DOUT), D7.4 (DIN)
- new net: D1.2 (DOUT), D2.4 (DIN)
- new net: D35.2 (DOUT), D36.4 (DIN)
- new net: D31.2 (DOUT), D32.4 (DIN)
- new net: D30.2 (DOUT), D31.4 (DIN)
- new net: D41.2 (DOUT), D42.4 (DIN)
- new net: D13.2 (DOUT), D14.4 (DIN)
- new net: D12.2 (DOUT), D13.4 (DIN)
- new net: D29.2 (DOUT), D30.4 (DIN)
- new net: D10.4 (DIN), D9.2 (DOUT)
- new net: D8.2 (DOUT), D9.4 (DIN)
- new net: D37.2 (DOUT), D38.4 (DIN)
- new net: D36.2 (DOUT), D37.4 (DIN)
- new net: D11.2 (DOUT), D12.4 (DIN)
- new net: D16.2 (DOUT), D17.4 (DIN)
- new net: D5.2 (DOUT), D6.4 (DIN)
- new net: D4.2 (DOUT), D5.4 (DIN)
- new net: D18.2 (DOUT), D19.4 (DIN)
- new net: D17.2 (DOUT), D18.4 (DIN)
- new net: D38.2 (DOUT), D39.4 (DIN)
- new net: D10.2 (DOUT), D11.4 (DIN)
- new net 5VLED: D1.4 (DIN), U9.3
- new net SELX: U1.10 (E6), U10.11 (A)
- new net SELY: U1.11 (B4), U10.10 (B)
- new net SELZ: U1.12 (B5), U10.9 (C)
- no-connect marks 0 -> 1
Other:
- moved on the sheet: C1, C10, C11, C12, C13, C14, C15, C16, C17, C18, C19, C2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

Commit message: Update PCB and schematic
Parts:
- D1, D13, D14, D15, D16, D17, D18, D2, D25, D26, D27, D28, D29, D3, D30, D37, D38, D39, D4, D40, D41, D42, D5, D6: footprint SkeletonKBD-Parts:SK6812MINI-E_nusumi -> project-specific-library:SK6812MINI-E_nusumi
- D10, D11, D12, D19, D20, D21, D22, D23, D24, D31, D32, D33, D34, D35, D36, D7, D8, D9: footprint SkeletonKBD-Parts:SK6812MINI-E_nusumi -> project-specific-library:SK6812MINI-E_nusumi_Rotated
- S39, S40: footprint project-specific-library:HE-Switch-2U_V -> project-specific-library:HE-Switch-2U
Changed lines of the file:
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@@
 			)
 		)
-		(property "Footprint" "SkeletonKBD-Parts:SK6812MINI-E_nusumi"
+		(property "Footprint" "project-specific-library:SK6812MINI-E_nusumi_Rotated"
 			(at 365.76 204.47 0)
 			(effects
@@
 			)
 		)
-		(property "Footprint" "SkeletonKBD-Parts:SK6812MINI-E_nusumi"
+		(property "Footprint" "project-specific-library:SK6812MINI-E_nusumi_Rotated"
 			(at 350.52 204.47 0)
 			(effects
@@
 			)
 		)
-		(property "Footprint" "SkeletonKBD-Parts:SK6812MINI-E_nusumi"
+		(property "Footprint" "project-specific-library:SK6812MINI-E_nusumi_Rotated"
 			(at 335.28 160.02 0)
 			(effects
@@
 			)
 		)
-		(property "Footprint" "SkeletonKBD-Parts:SK6812MINI-E_nusumi"
+		(property "Footprint" "project-specific-library:SK6812MINI-E_nusumi"
 			(at 314.96 204.47 0)
 			(effects
@@
 			)
 		)
-		(property "Footprint" "project-specific-library:HE-Switch-2U_V"
+		(property "Footprint" "project-specific-library:HE-Switch-2U"
 			(at 275.59 85.598 0)
 			(effects
@@
 			)
 		)
-		(property "Footprint" "SkeletonKBD-Parts:SK6812MINI-E_nusumi"
+		(property "Footprint" "project-specific-library:SK6812MINI-E_nusumi_Rotated"
 			(at 350.52 160.02 0)
 			(effects
@@
 			)
 		)
-		(property "Footprint" "SkeletonKBD-Parts:SK6812MINI-E_nusumi"
+		(property "Footprint" "project-specific-library:SK6812MINI-E_nusumi"
 			(at 345.44 118.11 0)
 			(effects
@@
 			)
 		)
-		(property "Footprint" "SkeletonKBD-Parts:SK6812MINI-E_nusumi"
+		(property "Footprint" "project-specific-library:SK6812MINI-E_nusumi_Rotated"
 			(at 381 160.02 0)
 			(effects
@@
 			)
 		)
-		(property "Footprint" "SkeletonKBD-Parts:SK6812MINI-E_nusumi"
+		(property "Footprint" "project-specific-library:SK6812MINI-E_nusumi"
 			(at 360.68 204.47 0)
 			(effects
@@
 			)
 		)
-		(property "Footprint" "project-specific-library:HE-Switch-2U_V"
+		(property "Footprint" "project-specific-library:HE-Switch-2U"
 			(at 275.59 108.458 0)
 			(effects
@@
 			)
 		)
-		(property "Footprint" "SkeletonKBD-Parts:SK6812MINI-E_nusumi"
+		(property "Footprint" "project-specific-library:SK6812MINI-E_nusumi"
 			(at 345.44 160.02 0)
 			(effects
@@
 			)
 		)
-		(property "Footprint" "SkeletonKBD-Parts:SK6812MINI-E_nusumi"
+		(property "Footprint" "project-specific-library:SK6812MINI-E_nusumi"
 			(at 330.2 204.47 0)
 			(effects
@@
 			)
 		)
-		(property "Footprint" "SkeletonKBD-Parts:SK6812MINI-E_nusumi"
+		(property "Footprint" "project-specific-library:SK6812MINI-E_nusumi"
 			(at 360.68 248.92 0)
 			(effects
@@
 			)
 		)
-		(property "Footprint" "SkeletonKBD-Parts:SK6812MINI-E_nusumi"
+		(property "Footprint" "project-specific-library:SK6812MINI-E_nusumi_Rotated"
 			(at 396.24 118.11 0)
 			(effects
@@
 			)
 		)
-		(property "Footprint" "SkeletonKBD-Parts:SK6812MINI-E_nusumi"
+		(property "Footprint" "project-specific-library:SK6812MINI-E_nusumi"
 			(at 330.2 118.11 0)
 			(effects
@@
 			)
 		)
-		(property "Footprint" "SkeletonKBD-Parts:SK6812MINI-E_nusumi"
+		(property "Footprint" "project-specific-library:SK6812MINI-E_nusumi_Rotated"
 			(at 335.28 204.47 0)
 			(effects
@@
 			)
 		)
-		(property "Footprint" "SkeletonKBD-Parts:SK6812MINI-E_nusumi"
+		(property "Footprint" "project-specific-library:SK6812MINI-E_nusumi_Rotated"
 			(at 396.24 204.47 0)
 			(effects
@@
 			)
 		)
-		(property "Footprint" "SkeletonKBD-Parts:SK6812MINI-E_nusumi"
+		(property "Footprint" "project-specific-library:SK6812MINI-E_nusumi"
 			(at 375.92 248.92 0)
 			(effects
@@
 			)
 		)
-		(property "Footprint" "SkeletonKBD-Parts:SK6812MINI-E_nusumi"
+		(property "Footprint" "project-specific-library:SK6812MINI-E_nusumi"
 			(at 314.96 160.02 0)
 			(effects
@@
 			)
 		)
-		(property "Footprint" "SkeletonKBD-Parts:SK6812MINI-E_nusumi"
+		(property "Footprint" "project-specific-library:SK6812MINI-E_nusumi"
 			(at 391.16 204.47 0)
 			(effects
@@
 			)
 		)
-		(property "Footprint" "SkeletonKBD-Parts:SK6812MINI-E_nusumi"
+		(property "Footprint" "project-specific-library:SK6812MINI-E_nusumi"
 			(at 375.92 204.47 0)
 			(effects
@@
 			)
 		)
-		(property "Footprint" "SkeletonKBD-Parts:SK6812MINI-E_nusumi"
+		(property "Footprint" "project-specific-library:SK6812MINI-E_nusumi_Rotated"
 			(at 365.76 118.11 0)
 			(effects
@@
 			)
 		)
-		(property "Footprint" "SkeletonKBD-Parts:SK6812MINI-E_nusumi"
+		(property "Footprint" "project-specific-library:SK6812MINI-E_nusumi"
 			(at 314.96 248.92 0)
 			(effects
@@
 			)
 		)
-		(property "Footprint" "SkeletonKBD-Parts:SK6812MINI-E_nusumi"
+		(property "Footprint" "project-specific-library:SK6812MINI-E_nusumi_Rotated"
 			(at 320.04 118.11 0)
 			(effects
@@
 			)
 		)
-		(property "Footprint" "SkeletonKBD-Parts:SK6812MINI-E_nusumi"
+		(property "Footprint" "project-specific-library:SK6812MINI-E_nusumi"
 			(at 360.68 160.02 0)
 			(effects
@@
 			)
 		)
-		(property "Footprint" "SkeletonKBD-Parts:SK6812MINI-E_nusumi"
+		(property "Footprint" "project-specific-library:SK6812MINI-E_nusumi"
 			(at 375.92 118.11 0)
 			(effects
@@
 			)
 		)
-		(property "Footprint" "SkeletonKBD-Parts:SK6812MINI-E_nusumi"
+		(property "Footprint" "project-specific-library:SK6812MINI-E_nusumi"
 			(at 314.96 118.11 0)
 			(effects
@@
 			)
 		)
-		(property "Footprint" "SkeletonKBD-Parts:SK6812MINI-E_nusumi"
+		(property "Footprint" "project-specific-library:SK6812MINI-E_nusumi_Rotated"
 			(at 396.24 160.02 0)
 			(effects
@@
 			)
 		)
-		(property "Footprint" "SkeletonKBD-Parts:SK6812MINI-E_nusumi"
+		(property "Footprint" "project-specific-library:SK6812MINI-E_nusumi_Rotated"
 			(at 381 204.47 0)
 			(effects
@@
 			)
 		)
-		(property "Footprint" "SkeletonKBD-Parts:SK6812MINI-E_nusumi"
+		(property "Footprint" "project-specific-library:SK6812MINI-E_nusumi"
 			(at 375.92 160.02 0)
 			(effects
@@
 			)
 		)
-		(property "Footprint" "SkeletonKBD-Parts:SK6812MINI-E_nusumi"
+		(property "Footprint" "project-specific-library:SK6812MINI-E_nusumi"
 			(at 345.44 248.92 0)
 			(effects
@@
 			)
 		)
-		(property "Footprint" "SkeletonKBD-Parts:SK6812MINI-E_nusumi"
+		(property "Footprint" "project-specific-library:SK6812MINI-E_nusumi_Rotated"
 			(at 320.04 204.47 0)
 			(effects
@@
 			)
 		)
-		(property "Footprint" "SkeletonKBD-Parts:SK6812MINI-E_nusumi"
+		(property "Footprint" "project-specific-library:SK6812MINI-E_nusumi_Rotated"
 			(at 365.76 160.02 0)
 			(effects
@@
 			)
 		)
-		(property "Footprint" "SkeletonKBD-Parts:SK6812MINI-E_nusumi"
+		(property "Footprint" "project-specific-library:SK6812MINI-E_nusumi"
 			(at 391.16 160.02 0)
 			(effects
@@
 			)
 		)
-		(property "Footprint" "SkeletonKBD-Parts:SK6812MINI-E_nusumi"
+		(property "Footprint" "project-specific-library:SK6812MINI-E_nusumi_Rotated"
 			(at 335.28 118.11 0)
 			(effects
@@
 			)
 		)
-		(property "Footprint" "SkeletonKBD-Parts:SK6812MINI-E_nusumi"
+		(property "Footprint" "project-specific-library:SK6812MINI-E_nusumi"
 			(at 330.2 160.02 0)
 			(effects
@@
 			)
 		)
-		(property "Footprint" "SkeletonKBD-Parts:SK6812MINI-E_nusumi"
+		(property "Footprint" "project-specific-library:SK6812MINI-E_nusumi_Rotated"
 			(at 381 118.11 0)
 			(effects
@@
 			)
 		)
-		(property "Footprint" "SkeletonKBD-Parts:SK6812MINI-E_nusumi"
+		(property "Footprint" "project-specific-library:SK6812MINI-E_nusumi"
 			(at 330.2 248.92 0)
 			(effects
@@
 			)
 		)
-		(property "Footprint" "SkeletonKBD-Parts:SK6812MINI-E_nusumi"
+		(property "Footprint" "project-specific-library:SK6812MINI-E_nusumi"
 			(at 391.16 248.92 0)
 			(effects
@@
 			)
 		)
-		(property "Footprint" "SkeletonKBD-Parts:SK6812MINI-E_nusumi"
+		(property "Footprint" "project-specific-library:SK6812MINI-E_nusumi"
 			(at 345.44 204.47 0)
 			(effects
@@
 			)
 		)
-		(property "Footprint" "SkeletonKBD-Parts:SK6812MINI-E_nusumi"
+		(property "Footprint" "project-specific-library:SK6812MINI-E_nusumi"
 			(at 391.16 118.11 0)
 			(effects
@@
 			)
 		)
-		(property "Footprint" "SkeletonKBD-Parts:SK6812MINI-E_nusumi"
+		(property "Footprint" "project-specific-library:SK6812MINI-E_nusumi_Rotated"
 			(at 320.04 160.02 0)
 			(effects
@@
 			)
 		)
-		(property "Footprint" "SkeletonKBD-Parts:SK6812MINI-E_nusumi"
+		(property "Footprint" "project-specific-library:SK6812MINI-E_nusumi"
 			(at 360.68 118.11 0)
 			(effects
@@
 			)
 		)
-		(property "Footprint" "SkeletonKBD-Parts:SK6812MINI-E_nusumi"
+		(property "Footprint" "project-specific-library:SK6812MINI-E_nusumi_Rotated"
 			(at 350.52 118.11 0)
 			(effects
