File: hw/cover/TrueStrike42-cover.kicad_pcb (KiCad board)
At the start: 2 copper layers, 47.2 x 68.2 mm, 4 parts

Commit message: Update TrueStrike42-cover.kicad_pcb
Add ID location for cover
Other:
- board text added: "JLCJLCJLCJLC"
Changed lines of the file:
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@@
 		(layer "Edge.Cuts")
 	)
+	(gr_text "JLCJLCJLCJLC"
+		(at 148.66 141 -0)
+		(layer "B.SilkS")
+		(effects
+			(font
+				(size 0.8 0.8)
+				(thickness 0.1)
+			)
+			(justify bottom mirror)
+		)
+	)
 )
